File: Hardware/Basic/stuff-BASIC.brd (EAGLE design)
At the start: 38 x 38 mm, 52 parts, among them SW1 SWITCH.MOM, SW2 SWITCH.MOM, SW5 SWITCH.MOM, U2 NRF52832_MODULE_MDBT42, U4 PCF8523

Commit message: done until 22 min mark
Parts:
- moved SW1 29.7 mm to (32.0, 4.01)
- moved SW2 25.1 mm to (21.7, 4.09)
- moved C6 6.66 mm to (13.8, 2.51)
- moved R15 6.42 mm to (16.0, 2.49)
- moved LDO2 6.16 mm to (14.2, 7.11)
- moved R12 6.11 mm to (11.8, 4.90)
- moved R11 3.97 mm to (23.8, 12.4)
- moved C20 3.63 mm to (12.3, 11.4)
- moved D4 3.63 mm to (7.98, 6.27)
- moved D5 3.59 mm to (7.92, 4.14)
- moved CHRG2 3.54 mm to (15.4, 11.4)
- moved C5 3.32 mm to (11.0, 2.44)
- moved C21 3.08 mm to (19.1, 11.3)
Connections:
- net VBATT renamed VBAT
- removed net N$16: SW1.B1, SW1.B2
- removed net N$18: SW1.A1
- new net SW1: SW1.A1, SW2.A1, SW5.A1
- net GND: now also SW1.B1, SW1.B2, SW2.B1, SW2.B2, SW5.B1, SW5.B2

Commit message: fixed inconsistency errors
Parts:
- removed SW5: SWITCH.MOM, LinnesLab-Switches:TACTILE_SWITCH_SMD_6.2MM_TALL
- removed USB2: USB.MICRO-BIGGERPADS, LinnesLab-Connectors:USB-MICRO-01.BIGGERPADS
- added J1: FTDI_DEVICESMD, LinnesLab-Connectors:FTDI-SMD
Connections:
- removed net USB+: USB2.3
- removed net USB-: USB2.2
- new net RXD.NRF: J1.TXO
- new net TXD.NRF: J1.RXI
- net DTR: now also J1.DTR
- net GND: now also J1.CTS, J1.GND; no longer SW5.B1, SW5.B2, USB2.5
- net SW1: no longer SW5.A1
- net V_USB: now also J1.VCC; no longer USB2.1
Changed lines of the file:
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@@
 <attribute name="VALUE" x="12.319" y="7.8232" size="1.27" layer="27" rot="R90"/>
-</element>
-<element name="USB2" library="LinnesLab-Connectors" package="USB-MICRO-01.BIGGERPADS" value="USB.MICRO-BIGGERPADS" x="2.9972" y="6.9596" smashed="yes" rot="MR90">
-<attribute name="NAME" x="6.2484" y="3.302" size="0.6604" layer="26" rot="MR90"/>
-<attribute name="VALUE" x="5.715" y="3.81" size="0.6604" layer="28" rot="MR90"/>
 </element>
 <element name="R15" library="LinnesLab-Passives" package="R0603" package3d_urn="urn:adsk.eagle:package:15661944/2" value="100k" x="16.0274" y="2.4892" smashed="yes" rot="R90">
@@
 <attribute name="VALUE" x="21.7424" y="0.9144" size="0.6096" layer="27" ratio="20" align="top-center"/>
 </element>
-<element name="SW5" library="LinnesLab-Switches" package="TACTILE_SWITCH_SMD_6.2MM_TALL" value="SWITCH.MOM" x="3.8608" y="-21.6408" smashed="yes">
-<attribute name="NAME" x="3.8608" y="-18.4658" size="0.6096" layer="25" ratio="20" align="bottom-center"/>
-<attribute name="VALUE" x="3.8608" y="-24.8158" size="0.6096" layer="27" ratio="20" align="top-center"/>
-</element>
+<element name="J1" library="LinnesLab-Connectors" package="FTDI-SMD" value="FTDI_DEVICESMD" x="8.9154" y="-13.3604" smashed="yes"/>
 </elements>
 <signals>
@@
 <contactref element="R11" pad="1"/>
 <contactref element="C21" pad="1"/>
-<contactref element="USB2" pad="5"/>
 <contactref element="J2" pad="1"/>
 <contactref element="R14" pad="1"/>
@@
 <contactref element="SW2" pad="B1"/>
 <contactref element="SW2" pad="B2"/>
-<contactref element="SW5" pad="B1"/>
-<contactref element="SW5" pad="B2"/>
+<contactref element="J1" pad="CTS"/>
+<contactref element="J1" pad="GND"/>
 <wire x1="42.1132" y1="31.2674" x2="46.3552" y2="31.0764" width="0" layer="19" extent="1-1"/>
 <wire x1="40.8432" y1="31.2674" x2="42.1132" y2="31.2674" width="0" layer="19" extent="1-1"/>
@@
 <wire x1="14.0669" y1="11.43" x2="19.1008" y2="12.1276" width="0" layer="19" extent="1-1"/>
 <wire x1="12.2682" y1="12.2038" x2="14.0669" y2="11.43" width="0" layer="19" extent="1-1"/>
-<wire x1="10.414" y1="7.6082" x2="12.2682" y2="12.2038" width="0" layer="19" extent="1-1"/>
+<wire x1="12.8985" y1="7.112" x2="14.0669" y2="11.43" width="0" layer="19" extent="1-1"/>
+<wire x1="10.414" y1="7.6082" x2="12.8985" y2="7.112" width="0" layer="19" extent="1-1"/>
 <wire x1="7.2254" y1="9.0932" x2="10.414" y2="7.6082" width="0" layer="19" extent="1-1"/>
-<wire x1="4.5022" y1="8.2596" x2="7.2254" y2="9.0932" width="0" layer="19" extent="1-16"/>
 <wire x1="5.5254" y1="11.7856" x2="7.2254" y2="9.0932" width="0" layer="19" extent="1-1"/>
+<wire x1="17.7674" y1="6.3394" x2="12.8985" y2="7.112" width="0" layer="19" extent="1-1"/>
+<wire x1="16.0274" y1="1.6392" x2="17.7674" y2="6.3394" width="0" layer="19" extent="1-1"/>
+<wire x1="13.7668" y1="1.6646" x2="16.0274" y2="1.6392" width="0" layer="19" extent="1-1"/>
+<wire x1="10.9728" y1="1.5884" x2="13.7668" y2="1.6646" width="0" layer="19" extent="1-1"/>
+<wire x1="35.9536" y1="6.2632" x2="33.2396" y2="11.2574" width="0" layer="19" extent="1-16"/>
+<wire x1="36.6396" y1="1.1574" x2="35.9536" y2="6.2632" width="0" layer="19" extent="1-16"/>
 <wire x1="16.0158" y1="19.8566" x2="21.6052" y2="21.3614" width="0" layer="19" extent="1-1"/>
 <wire x1="14.6158" y1="19.8566" x2="16.0158" y2="19.8566" width="0" layer="19" extent="1-1"/>
@@
 <wire x1="8.3158" y1="19.8566" x2="8.5514" y2="24.4094" width="0" layer="19" extent="1-1"/>
 <wire x1="12.1548" y1="29.9212" x2="12.4968" y2="24.2974" width="0" layer="19" extent="1-1"/>
+<wire x1="25.7174" y1="6.3394" x2="24.6498" y2="12.4206" width="0" layer="19" extent="1-1"/>
+<wire x1="28.0036" y1="6.2632" x2="25.7174" y2="6.3394" width="0" layer="19" extent="1-1"/>
 <wire x1="2.413" y1="17.1704" x2="5.5254" y2="11.7856" width="0" layer="19" extent="1-1"/>
-<wire x1="12.8985" y1="7.112" x2="14.0669" y2="11.43" width="0" layer="19" extent="1-1"/>
-<wire x1="10.9728" y1="1.5884" x2="12.8985" y2="7.112" width="0" layer="19" extent="1-1"/>
-<wire x1="13.7668" y1="1.6646" x2="12.8985" y2="7.112" width="0" layer="19" extent="1-1"/>
-<wire x1="16.0274" y1="1.6392" x2="13.7668" y2="1.6646" width="0" layer="19" extent="1-1"/>
 <wire x1="26.0832" y1="32.0194" x2="28.1178" y2="25.1324" width="0" layer="19" extent="1-1"/>
-<wire x1="35.9536" y1="6.2632" x2="10.9728" y2="1.5884" width="0" layer="19" extent="1-1"/>
-<wire x1="28.0036" y1="6.2632" x2="35.9536" y2="6.2632" width="0" layer="19" extent="1-1"/>
-<wire x1="17.7674" y1="6.3394" x2="28.0036" y2="6.2632" width="0" layer="19" extent="1-1"/>
-<wire x1="25.7174" y1="6.3394" x2="17.7674" y2="6.3394" width="0" layer="19" extent="1-1"/>
-<wire x1="-0.1142" y1="-19.3908" x2="17.7674" y2="6.3394" width="0" layer="19" extent="1-1"/>
-<wire x1="7.8358" y1="-19.3908" x2="-0.1142" y2="-19.3908" width="0" layer="19" extent="1-1"/>
-<wire x1="36.6396" y1="1.1574" x2="33.2396" y2="11.2574" width="0" layer="19" extent="16-16"/>
+<wire x1="15.2654" y1="-13.3604" x2="16.0274" y2="1.6392" width="0" layer="19" extent="1-1"/>
+<wire x1="12.7254" y1="-13.3604" x2="15.2654" y2="-13.3604" width="0" layer="19" extent="1-1"/>
 </signal>
 <signal name="N$4">
@@
 <signal name="DTR">
 <contactref element="C14" pad="1"/>
+<contactref element="J1" pad="DTR"/>
+<wire x1="2.5654" y1="-13.3604" x2="49.4792" y2="19.4174" width="0" layer="19" extent="1-1"/>
 </signal>
 <signal name="P0.10/NFC2">
@@
 </signal>
 <signal name="V_USB">
-<contactref element="USB2" pad="1"/>
 <contactref element="D5" pad="+"/>
-<wire x1="6.7748" y1="4.1402" x2="4.5022" y2="5.6596" width="0" layer="19" extent="1-16"/>
+<contactref element="J1" pad="VCC"/>
+<wire x1="10.1854" y1="-13.3604" x2="6.7748" y2="4.1402" width="0" layer="19" extent="1-1"/>
 </signal>
 <signal name="CHRG.STAT">
@@
 <contactref element="CHRG2" pad="1"/>
 <wire x1="10.9864" y1="4.9022" x2="14.0669" y2="12.38" width="0" layer="19" extent="1-1"/>
-</signal>
-<signal name="USB-">
-<contactref element="USB2" pad="2"/>
-</signal>
-<signal name="USB+">
-<contactref element="USB2" pad="3"/>
 </signal>
 <signal name="BATT">
@@
 <contactref element="SW1" pad="A1"/>
 <contactref element="SW2" pad="A1"/>
-<contactref element="SW5" pad="A1"/>
-<wire x1="17.7674" y1="1.8394" x2="-0.1142" y2="-23.8908" width="0" layer="19" extent="1-1"/>
-<wire x1="28.0036" y1="1.7632" x2="17.7674" y2="1.8394" width="0" layer="19" extent="1-1"/>
+<wire x1="17.7674" y1="1.8394" x2="28.0036" y2="1.7632" width="0" layer="19" extent="1-1"/>
 </signal>
 <signal name="VBAT">
 <contactref element="U4" pad="3"/>
 </signal>
+<signal name="TXD.NRF">
+<contactref element="J1" pad="RXI"/>
+</signal>
+<signal name="RXD.NRF">
+<contactref element="J1" pad="TXO"/>
+</signal>
 </signals>

Commit message: Complete schematic
Parts:
- removed C10, C11: 300p, LinnesLab-Passives:C0603
Connections:
- removed net RXD: U2.21
- removed net TXD: U2.19
- new net A4/PPG: U2.5
- new net A5/TIA: U2.6
- new net A7/BATT: U2.8
- new net D11/SW1: U2.25
- new net D15/SW2: U2.29
- new net D16/CS.OLED: U2.30
- new net D27/CHRG.STATUS: U2.4
- new net D3/RESET.OLED: U2.16
- new net D30/LED.CNTRL: U2.7
- new net D4/DC.OLED: U2.17
- new net D5/CD1: U2.18
- new net D7/SD.CS: U2.20
- net GND: no longer C10.2, C11.2
- net P0.09/NFC1: no longer C11.1
- net P0.10/NFC2: no longer C10.1
- net RXD.NRF: now also U2.21
- net TXD.NRF: now also U2.19
Changed lines of the file:
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@@
 <attribute name="VALUE" x="28.7782" y="13.3604" size="0.7112" layer="27"/>
-</element>
-<element name="C10" library="LinnesLab-Passives" package="C0603" package3d_urn="urn:adsk.eagle:package:15661989/2" value="300p" x="34.7472" y="15.9004" smashed="yes">
-<attribute name="NAME" x="34.1122" y="16.5354" size="0.7112" layer="25"/>
-<attribute name="VALUE" x="34.1122" y="13.9954" size="0.7112" layer="27"/>
-</element>
-<element name="C11" library="LinnesLab-Passives" package="C0603" package3d_urn="urn:adsk.eagle:package:15661989/2" value="300p" x="34.3662" y="18.0594" smashed="yes">
-<attribute name="NAME" x="33.7312" y="18.6944" size="0.7112" layer="25"/>
-<attribute name="VALUE" x="33.7312" y="16.1544" size="0.7112" layer="27"/>
 </element>
 <element name="C12" library="LinnesLab-Passives" package="C0805" package3d_urn="urn:adsk.eagle:package:15662010/2" value="10u" x="22.5552" y="21.3614" smashed="yes">
@@
 <contactref element="C8" pad="1"/>
 <contactref element="C9" pad="2"/>
-<contactref element="C11" pad="2"/>
-<contactref element="C10" pad="2"/>
 <contactref element="C12" pad="1"/>
 <contactref element="CORTEX1" pad="3"/>
@@
 <wire x1="43.3712" y1="24.6634" x2="43.6252" y2="26.9494" width="0" layer="19" extent="1-1"/>
 <wire x1="42.4432" y1="19.6464" x2="43.3712" y2="24.6634" width="0" layer="19" extent="1-1"/>
-<wire x1="35.2162" y1="18.0594" x2="42.4432" y2="19.6464" width="0" layer="19" extent="1-1"/>
-<wire x1="35.5972" y1="15.9004" x2="35.2162" y2="18.0594" width="0" layer="19" extent="1-1"/>
-<wire x1="35.7396" y1="14.3574" x2="35.5972" y2="15.9004" width="0" layer="19" extent="1-16"/>
-<wire x1="34.8832" y1="20.5694" x2="35.2162" y2="18.0594" width="0" layer="19" extent="1-1"/>
+<wire x1="34.8832" y1="20.5694" x2="42.4432" y2="19.6464" width="0" layer="19" extent="1-1"/>
+<wire x1="35.7396" y1="14.3574" x2="34.8832" y2="20.5694" width="0" layer="19" extent="1-16"/>
 <wire x1="33.2396" y1="11.2574" x2="35.7396" y2="14.3574" width="0" layer="19" extent="16-16"/>
 <wire x1="30.2632" y1="15.2654" x2="33.2396" y2="11.2574" width="0" layer="19" extent="1-16"/>
@@
 </signal>
 <signal name="P0.09/NFC1">
-<contactref element="C11" pad="1"/>
 <contactref element="U2" pad="22"/>
-<wire x1="33.5162" y1="18.0594" x2="33.4832" y2="20.5694" width="0" layer="19" extent="1-1"/>
 </signal>
 <signal name="DTR">
@@
 </signal>
 <signal name="P0.10/NFC2">
-<contactref element="C10" pad="1"/>
 <contactref element="U2" pad="23"/>
-<wire x1="33.8972" y1="15.9004" x2="34.1832" y2="20.5694" width="0" layer="19" extent="1-1"/>
 </signal>
 <signal name="DFU">
@@
 <contactref element="SD3" pad="7"/>
 <wire x1="32.8396" y1="12.3574" x2="35.2832" y2="24.1194" width="0" layer="19" extent="1-16"/>
-</signal>
-<signal name="RXD">
-<contactref element="U2" pad="21"/>
-</signal>
-<signal name="TXD">
-<contactref element="U2" pad="19"/>
 </signal>
 <signal name="FRST">
@@
 <signal name="TXD.NRF">
 <contactref element="J1" pad="RXI"/>
+<contactref element="U2" pad="19"/>
+<wire x1="7.6454" y1="-13.3604" x2="31.3832" y2="20.5694" width="0" layer="19" extent="1-1"/>
 </signal>
 <signal name="RXD.NRF">
 <contactref element="J1" pad="TXO"/>
+<contactref element="U2" pad="21"/>
+<wire x1="5.1054" y1="-13.3604" x2="32.7832" y2="20.5694" width="0" layer="19" extent="1-1"/>
+</signal>
+<signal name="D27/CHRG.STATUS">
+<contactref element="U2" pad="4"/>
+</signal>
+<signal name="A4/PPG">
+<contactref element="U2" pad="5"/>
+</signal>
+<signal name="A5/TIA">
+<contactref element="U2" pad="6"/>
+</signal>
+<signal name="D30/LED.CNTRL">
+<contactref element="U2" pad="7"/>
+</signal>
+<signal name="A7/BATT">
+<contactref element="U2" pad="8"/>
+</signal>
+<signal name="D16/CS.OLED">
+<contactref element="U2" pad="30"/>
+</signal>
+<signal name="D15/SW2">
+<contactref element="U2" pad="29"/>
+</signal>
+<signal name="D11/SW1">
+<contactref element="U2" pad="25"/>
+</signal>
+<signal name="D3/RESET.OLED">
+<contactref element="U2" pad="16"/>
+</signal>
+<signal name="D4/DC.OLED">
+<contactref element="U2" pad="17"/>
+</signal>
+<signal name="D5/CD1">
+<contactref element="U2" pad="18"/>
+</signal>
+<signal name="D7/SD.CS">
+<contactref element="U2" pad="20"/>
 </signal>
 </signals>

Commit message: Start organizing and routing
Parts:
- removed SD3: (no value), LinnesLab-Connectors:MICROSD
- added J3: (no value), LinnesLab-Connectors:1X07_1.27MM
- moved C12 39.9 mm to (-14.9, 35.2)
- moved C13 39.9 mm to (-27.7, 37.4)
- moved C15 39.9 mm to (-26.3, 37.5)
- moved C16 39.9 mm to (-9.35, 38.1)
- moved C17 39.9 mm to (-23.6, 37.5)
- moved C18 39.9 mm to (-10.9, 37.8)
- moved C19 39.9 mm to (-25.0, 37.5)
- moved C2 39.9 mm to (-24.5, 43.8)
- moved C20 39.9 mm to (-25.2, 25.2)
- moved C21 39.9 mm to (-18.4, 25.1)
- moved C5 39.9 mm to (-26.5, 16.3)
- moved C6 39.9 mm to (-23.7, 16.4)
- moved C7 39.9 mm to (-13.8, 39.1)
- moved C9 39.9 mm to (-8.05, 29.1)
- moved CHRG2 39.9 mm to (-22.1, 25.3)
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Connections:
- net VBAT renamed VBATT
- removed net BATT: R13.1, R14.2
- removed net CD1: SD3.CD1
- removed net CD2: SD3.CD2
- removed net CHRG.STAT: CHRG2.1, R12.1
- removed net CS.OLED: U3.13
- removed net D30/LED.CNTRL: U2.7
- removed net DC.OLED: U3.15
- removed net RESET.OLED: U3.14
- removed net SD.CS: SD3.2
- removed net SW1: SW1.A1, SW2.A1
- new net D30/LED.CTRL: J3.5, U2.7
- new net N$16: J3.4
- net 3.3V: no longer SD3.4
- net A4/PPG: now also J3.7
- net A5/TIA: now also J3.6
- net A7/BATT: now also R13.1, R14.2
- net D11/SW1: now also SW1.A1
- net D15/SW2: now also SW2.A1
- net D16/CS.OLED: now also U3.13
- net D27/CHRG.STATUS: now also CHRG2.1, R12.1
- net D3/RESET.OLED: now also U3.14
- net D4/DC.OLED: now also U3.15
- net GND: now also J3.3; no longer SD3.6, SD3.MT1, SD3.MT2
- net MISO: no longer SD3.7
- net MOSI: no longer SD3.3
- net SCK: no longer SD3.5
- net SCL: now also J3.2
- net SDA: now also J3.1
Routing:
- net RESET: track 0.00 -> 8.71 mm, vias 0 -> 1
- net LED2: track 0.00 -> 7.88 mm
- net LED1: track 0.00 -> 5.24 mm
- net GND: track 0.00 -> 3.31 mm, vias 0 -> 1
- net N$9: track 0.00 -> 1.95 mm
- net N$10: track 0.00 -> 1.88 mm
- added copper zone on layer 1, net 3.3V
- added copper zone on layer 16, net GND

Commit message: Airwires
Parts:
- removed C2: 1u, LinnesLab-Passives:C0603
- removed R15: 100k, LinnesLab-Passives:R0603
- removed U4: PCF8523, LinnesLab-Clocks:SO8
- removed XTAL3: 32.7680kHz, LinnesLab-Clocks:2-SMD.NOLEAD.2.0MMTO1.2MM
- added C3: 1u, LinnesLab-Passives:C0603
- added U5: PCF8523, LinnesLab-Clocks:SO8
- added XTAL4: 32.7680kHz, LinnesLab-Clocks:2-SMD.NOLEAD.2.0MMTO1.2MM
- C13, C15, C17, C18, C19: device LinnesLab-Passives:C0402 -> LinnesLab-Passives:C0603
- moved R7 62.0 mm to (30.7, 18.1), turned to 270 degrees
- moved C18 47.5 mm to (32.2, 18.1)
- moved R6 45.1 mm to (13.8, 22.3), turned to 270 degrees
- moved C16 43.4 mm to (29.2, 18.1), turned to 90 degrees
- moved C17 39.0 mm to (12.2, 22.1)
- moved C19 38.7 mm to (10.6, 22.2)
- moved C20 38.6 mm to (9.30, 7.90), turned to 180 degrees
- moved C15 38.5 mm to (9.04, 22.2), turned to 270 degrees
- moved C13 38.3 mm to (7.44, 22.1), turned to 270 degrees
- moved R12 37.6 mm to (8.64, 3.20), turned to 180 degrees
- moved CHRG2 37.0 mm to (9.07, 5.38), turned to 90 degrees
- moved L2 36.0 mm to (17.8, 26.4), turned to 0 degrees
- moved D5 34.0 mm to (3.68, 10.9), turned to 270 degrees
- moved C7 33.3 mm to (17.7, 28.2), turned to 180 degrees
- moved C12 33.1 mm to (17.8, 30.3), turned to 358.7 degrees
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Connections:
- removed net N$16: J3.4
- removed net N$19: U4.2, XTAL3.P$1
- removed net N$20: U4.1, XTAL3.P$2
- new net N$21: U5.2, XTAL4.P$1
- new net N$22: U5.1, XTAL4.P$2
- net 3.3V: now also C3.1, J3.4, U5.8; no longer C2.1, R15.2, U4.8
- net GND: now also C3.2, U5.4; no longer C2.2, R15.1, SW1.B1, SW2.B1, U4.4
- net SCL: now also U5.6; no longer U4.6
- net SDA: now also U5.5; no longer U4.5
- net VBATT: now also U5.3; no longer U4.3
Routing:
- net GND: track 3.31 -> 56.4 mm, vias 1 -> 24
- net D27/CHRG.STATUS: track 0.00 -> 32.5 mm, vias 0 -> 2
- net SCL: track 0.00 -> 31.2 mm
- net SDA: track 0.00 -> 30.3 mm, vias 0 -> 1
- net A7/BATT: track 0.00 -> 27.1 mm
- net DTR: track 0.00 -> 22.5 mm, vias 0 -> 1
- net D15/SW2: track 0.00 -> 21.8 mm, vias 0 -> 2
- net RXD.NRF: track 0.00 -> 21.3 mm, vias 0 -> 1
- net TXD.NRF: track 0.00 -> 20.6 mm, vias 0 -> 1
- net D11/SW1: track 0.00 -> 19.7 mm, vias 0 -> 2
- net D16/CS.OLED: track 0.00 -> 19.3 mm, vias 0 -> 2
- net VLIPO: track 0.00 -> 19.3 mm
- net RESET: track 8.71 -> 27.9 mm, vias 1 -> 3
- net SCK: track 0.00 -> 16.9 mm, vias 0 -> 2
- net MOSI: track 0.00 -> 16.4 mm, vias 0 -> 2
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